Commit message: Update f450.urdf

File: f450/urdf/f450.urdf (robot description, URDF)
Before this commit: robot f450, 14 links, 13 joints
Links:
- link back_arm_link: mass 0.084665 -> None; geometry visual mesh filename=package://f450/meshes/back_arm_link.STL
- link base_link: mass 0.37844186203839 -> None; geometry visual mesh filename=package://f450/meshes/base_link.STL
- link battery_link: mass 0.19453 -> None; geometry visual mesh filename=package://f450/meshes/battery_link.STL
- link d435_link: mass 0.043919 -> None; geometry visual mesh filename=package://f450/meshes/d435_link.STL
- link front_arm_link: mass 0.084665 -> None; geometry visual mesh filename=package://f450/meshes/front_arm_link.STL
- link jetson_link: mass 0.49209 -> None; geometry visual mesh filename=package://f450/meshes/jetson_link.STL
- link leg_link: mass 0.0540891840555198 -> None; geometry visual mesh filename=package://f450/meshes/leg_link.STL
- link motor_link: mass 0.057143 -> None; geometry visual mesh filename=package://f450/meshes/motor_link.STL
- link prop_guard_link: mass 0.084635 -> None; geometry visual mesh filename=package://f450/meshes/prop_guard_link.STL
- link rotor1: mass 0.01285 -> None; geometry visual mesh filename=package://f450/meshes/rotor1.STL
- link rotor2: mass 0.014286 -> None; geometry visual mesh filename=package://f450/meshes/rotor1.STL
- link rotor3: mass 0.014286 -> None; geometry visual mesh filename=package://f450/meshes/rotor1.STL
- link rotor4: mass 0 -> None; geometry visual mesh filename=package://f450/meshes/rotor1.STL
- link t265_link: mass 0.02522 -> None; geometry visual mesh filename=package://f450/meshes/t265_link.STL
Joints:
- removed joint leg_link_join
- added joint leg_link_joint: type fixed, parent base_link, child leg_link, origin xyz=0 0 0.132 rpy=0 0 0, axis 0 0 0
